File: 2225/PE01/2225_PE01.kicad_sch (KiCad schematic)
At the start: 90 parts, among them J1 Screw_Terminal_01x03, J2 Screw_Terminal_01x03, J3 Screw_Terminal_01x02

Commit message: Connected P800 (DC supply) to PE01 tone board, audio source to PE01, and PE01 to dummy P700 main amplifier. Changed some hierarchical label names in multiple schematics.
Parts:
- CE1, CE2: value 0.22u -> (none); footprint Capacitor_THT:C_Rect_L16.5mm_W4.7mm_P15.00mm_MKT -> (none)
- CE10, CE9: value 2200p -> (none); footprint Capacitor_THT:C_Rect_L7.2mm_W3.5mm_P5.00mm_FKS2_FKP2_MKS2_MKP2 -> (none)
- CE11, CE12: value 6800p -> (none); footprint Capacitor_THT:C_Rect_L7.2mm_W3.5mm_P5.00mm_FKS2_FKP2_MKS2_MKP2 -> (none)
- CE13, CE14, CE15, CE16: value 0.022u -> (none); footprint Capacitor_THT:C_Rect_L10.0mm_W4.0mm_P7.50mm_FKS3_FKP3 -> (none)
- CE17, CE18: value 0.01u -> (none); footprint Capacitor_THT:C_Rect_L9.0mm_W3.2mm_P7.50mm_MKT -> (none)
- CE19, CE20: value 1u -> (none); footprint Capacitor_THT:CP_Radial_D5.0mm_P2.50mm -> (none)
- CE21, CE22: value 3.3u -> (none); footprint Capacitor_THT:CP_Radial_D6.3mm_P2.50mm -> (none)
- CE23: value 1u -> (none); footprint Capacitor_THT:C_Radial_D6.3mm_H11.0mm_P3.50mm -> (none)
- CE24: value 1u -> (none); footprint Capacitor_THT:C_Radial_D6.3mm_H11.0mm_P2.50mm -> (none)
- CE25: value 220u -> (none); footprint Capacitor_THT:CP_Radial_D10.0mm_P5.00mm -> (none)
- CE3, CE4: value 10u -> (none); footprint Capacitor_THT:CP_Radial_D6.3mm_P2.50mm -> (none)
- CE5, CE6: value 4.7u -> (none); footprint Capacitor_THT:CP_Radial_D5.0mm_P2.50mm -> (none)
- CE7, CE8: value 100p -> (none); footprint Capacitor_THT:C_Disc_D7.0mm_W2.5mm_P5.00mm -> (none)
- HE1, HE2, HE5, HE6: value KSC1845FTA -> (none); footprint Package_TO_SOT_THT:TO-92_Inline -> (none)
- HE3, HE4, HE7, HE8: value KSA992FTA -> (none); footprint Package_TO_SOT_THT:TO-92_Inline -> (none)
- J1, J2: footprint Connector_Molex:Molex_Eurostyle_39357-0003_1x03_P3.5mm_Horizontal -> (none)
- J3: footprint Connector_Molex:Molex_Eurostyle_39357-0002_1x02_P3.5mm_Horizontal -> (none)
- RE1, RE17, RE18, RE2, RE35, RE36, RE49, RE50: value 470k -> (none); footprint Resistor_THT:R_Axial_DIN0309_L9.0mm_D3.2mm_P12.70mm_Horizontal -> (none)
- RE10, RE29, RE30, RE37, RE38, RE9: value 27k -> (none); footprint Resistor_THT:R_Axial_DIN0309_L9.0mm_D3.2mm_P12.70mm_Horizontal -> (none)
- RE11: value 1k -> (none); footprint Resistor_THT:R_Axial_DIN0309_L9.0mm_D3.2mm_P20.32mm_Horizontal -> (none)
- RE12, RE15, RE16: value 1k -> (none); footprint Resistor_THT:R_Axial_DIN0309_L9.0mm_D3.2mm_P12.70mm_Horizontal -> (none)
- RE13, RE14: value 7.5k -> (none); footprint Resistor_THT:R_Axial_DIN0309_L9.0mm_D3.2mm_P12.70mm_Horizontal -> (none)
- RE19, RE20, RE25, RE26, RE27, RE28: value 5.6k -> (none); footprint Resistor_THT:R_Axial_DIN0309_L9.0mm_D3.2mm_P12.70mm_Horizontal -> (none)
- RE21, RE22, RE31, RE32: value 12k -> (none); footprint Resistor_THT:R_Axial_DIN0309_L9.0mm_D3.2mm_P12.70mm_Horizontal -> (none)
- RE23, RE24: value 150k -> (none); footprint Resistor_THT:R_Axial_DIN0309_L9.0mm_D3.2mm_P12.70mm_Horizontal -> (none)
- RE3, RE4: value 390 -> (none); footprint Resistor_THT:R_Axial_DIN0309_L9.0mm_D3.2mm_P12.70mm_Horizontal -> (none)
- RE33, RE34: value 15k -> (none); footprint Resistor_THT:R_Axial_DIN0309_L9.0mm_D3.2mm_P12.70mm_Horizontal -> (none)
- RE39, RE40: value 2.2meg -> (none); footprint Resistor_THT:R_Axial_DIN0309_L9.0mm_D3.2mm_P12.70mm_Horizontal -> (none)
- RE41, RE42: value 68k -> (none); footprint Resistor_THT:R_Axial_DIN0309_L9.0mm_D3.2mm_P12.70mm_Horizontal -> (none)
- RE43, RE44: value 47k -> (none); footprint Resistor_THT:R_Axial_DIN0309_L9.0mm_D3.2mm_P12.70mm_Horizontal -> (none)
- RE45, RE46, RE8: value 10k -> (none); footprint Resistor_THT:R_Axial_DIN0309_L9.0mm_D3.2mm_P12.70mm_Horizontal -> (none)
- RE47, RE48: value 220 -> (none); footprint Resistor_THT:R_Axial_DIN0309_L9.0mm_D3.2mm_P12.70mm_Horizontal -> (none)
- RE5, RE6: value 1meg -> (none); footprint Resistor_THT:R_Axial_DIN0309_L9.0mm_D3.2mm_P5.08mm_Vertical -> (none)
- RE51, RE52, RE53: value 100k -> (none); footprint Potentiometer_THT:Potentiometer_Marantz_RM0104005 -> (none)
- RE54: value 820 -> (none); footprint Resistor_THT:R_Axial_DIN0309_L9.0mm_D3.2mm_P12.70mm_Horizontal -> (none)
- RE7: value 100k -> (none); footprint Resistor_THT:R_Axial_DIN0309_L9.0mm_D3.2mm_P12.70mm_Horizontal -> (none)
Connections:
- net V_power_in_35VDC renamed 35VDC
- net V_signal_in_L renamed L_in
- net V_signal_in_R renamed R_in
- net V_signal_out_L renamed L_out
- net V_signal_out_R renamed R_out

Commit message: Committing some changes to 2225_PE01.kicad_sch, but I dont really know why the file changed.
Parts:
- CE1, CE2: value (none) -> 0.22u; footprint (none) -> Capacitor_THT:C_Rect_L16.5mm_W4.7mm_P15.00mm_MKT
- CE10, CE9: value (none) -> 2200p; footprint (none) -> Capacitor_THT:C_Rect_L7.2mm_W3.5mm_P5.00mm_FKS2_FKP2_MKS2_MKP2
- CE11, CE12: value (none) -> 6800p; footprint (none) -> Capacitor_THT:C_Rect_L7.2mm_W3.5mm_P5.00mm_FKS2_FKP2_MKS2_MKP2
- CE13, CE14, CE15, CE16: value (none) -> 0.022u; footprint (none) -> Capacitor_THT:C_Rect_L10.0mm_W4.0mm_P7.50mm_FKS3_FKP3
- CE17, CE18: value (none) -> 0.01u; footprint (none) -> Capacitor_THT:C_Rect_L9.0mm_W3.2mm_P7.50mm_MKT
- CE19, CE20: value (none) -> 1u; footprint (none) -> Capacitor_THT:CP_Radial_D5.0mm_P2.50mm
- CE21, CE22: value (none) -> 3.3u; footprint (none) -> Capacitor_THT:CP_Radial_D6.3mm_P2.50mm
- CE23: value (none) -> 1u; footprint (none) -> Capacitor_THT:C_Radial_D6.3mm_H11.0mm_P3.50mm
- CE24: value (none) -> 1u; footprint (none) -> Capacitor_THT:C_Radial_D6.3mm_H11.0mm_P2.50mm
- CE25: value (none) -> 220u; footprint (none) -> Capacitor_THT:CP_Radial_D10.0mm_P5.00mm
- CE3, CE4: value (none) -> 10u; footprint (none) -> Capacitor_THT:CP_Radial_D6.3mm_P2.50mm
- CE5, CE6: value (none) -> 4.7u; footprint (none) -> Capacitor_THT:CP_Radial_D5.0mm_P2.50mm
- CE7, CE8: value (none) -> 100p; footprint (none) -> Capacitor_THT:C_Disc_D7.0mm_W2.5mm_P5.00mm
- HE1, HE2, HE5, HE6: value (none) -> KSC1845FTA; footprint (none) -> Package_TO_SOT_THT:TO-92_Inline
- HE3, HE4, HE7, HE8: value (none) -> KSA992FTA; footprint (none) -> Package_TO_SOT_THT:TO-92_Inline
- J1, J2: footprint (none) -> Connector_Molex:Molex_Eurostyle_39357-0003_1x03_P3.5mm_Horizontal
- J3: footprint (none) -> Connector_Molex:Molex_Eurostyle_39357-0002_1x02_P3.5mm_Horizontal
- RE1, RE17, RE18, RE2, RE35, RE36, RE49, RE50: value (none) -> 470k; footprint (none) -> Resistor_THT:R_Axial_DIN0309_L9.0mm_D3.2mm_P12.70mm_Horizontal
- RE10, RE29, RE30, RE37, RE38, RE9: value (none) -> 27k; footprint (none) -> Resistor_THT:R_Axial_DIN0309_L9.0mm_D3.2mm_P12.70mm_Horizontal
- RE11: value (none) -> 1k; footprint (none) -> Resistor_THT:R_Axial_DIN0309_L9.0mm_D3.2mm_P20.32mm_Horizontal
- RE12, RE15, RE16: value (none) -> 1k; footprint (none) -> Resistor_THT:R_Axial_DIN0309_L9.0mm_D3.2mm_P12.70mm_Horizontal
- RE13, RE14: value (none) -> 7.5k; footprint (none) -> Resistor_THT:R_Axial_DIN0309_L9.0mm_D3.2mm_P12.70mm_Horizontal
- RE19, RE20, RE25, RE26, RE27, RE28: value (none) -> 5.6k; footprint (none) -> Resistor_THT:R_Axial_DIN0309_L9.0mm_D3.2mm_P12.70mm_Horizontal
- RE21, RE22, RE31, RE32: value (none) -> 12k; footprint (none) -> Resistor_THT:R_Axial_DIN0309_L9.0mm_D3.2mm_P12.70mm_Horizontal
- RE23, RE24: value (none) -> 150k; footprint (none) -> Resistor_THT:R_Axial_DIN0309_L9.0mm_D3.2mm_P12.70mm_Horizontal
- RE3, RE4: value (none) -> 390; footprint (none) -> Resistor_THT:R_Axial_DIN0309_L9.0mm_D3.2mm_P12.70mm_Horizontal
- RE33, RE34: value (none) -> 15k; footprint (none) -> Resistor_THT:R_Axial_DIN0309_L9.0mm_D3.2mm_P12.70mm_Horizontal
- RE39, RE40: value (none) -> 2.2meg; footprint (none) -> Resistor_THT:R_Axial_DIN0309_L9.0mm_D3.2mm_P12.70mm_Horizontal
- RE41, RE42: value (none) -> 68k; footprint (none) -> Resistor_THT:R_Axial_DIN0309_L9.0mm_D3.2mm_P12.70mm_Horizontal
- RE43, RE44: value (none) -> 47k; footprint (none) -> Resistor_THT:R_Axial_DIN0309_L9.0mm_D3.2mm_P12.70mm_Horizontal
- RE45, RE46, RE8: value (none) -> 10k; footprint (none) -> Resistor_THT:R_Axial_DIN0309_L9.0mm_D3.2mm_P12.70mm_Horizontal
- RE47, RE48: value (none) -> 220; footprint (none) -> Resistor_THT:R_Axial_DIN0309_L9.0mm_D3.2mm_P12.70mm_Horizontal
- RE5, RE6: value (none) -> 1meg; footprint (none) -> Resistor_THT:R_Axial_DIN0309_L9.0mm_D3.2mm_P5.08mm_Vertical
- RE51, RE52, RE53: value (none) -> 100k; footprint (none) -> Potentiometer_THT:Potentiometer_Marantz_RM0104005
- RE54: value (none) -> 820; footprint (none) -> Resistor_THT:R_Axial_DIN0309_L9.0mm_D3.2mm_P12.70mm_Horizontal
- RE7: value (none) -> 100k; footprint (none) -> Resistor_THT:R_Axial_DIN0309_L9.0mm_D3.2mm_P12.70mm_Horizontal
