File: 2225/P800/P800.kicad_sch (KiCad schematic)
At the start: 28 parts, among them J1 Screw_Terminal_01x05, J2 Conn_Coaxial, J3 Conn_Coaxial, J4 Conn_Coaxial, J5 Conn_Coaxial

Commit message: Added footprints and 3D models for all components; assigned footprints to all components; populated PCB file with all footprints
Parts:
- added HS1: Heatsink_Pad, P800_footprint_library:heatsink_577202B04000G, symbol Mechanical:Heatsink_Pad
- C002, C003: footprint (none) -> P800_footprint_library:cap_electrolytic_A50
- C802: footprint (none) -> P800_footprint_library:cap_ceramic_RDER72H103K1M1H03A
- C803, C804: footprint (none) -> P800_footprint_library:cap_electrolytic_UKW1J471MHD1TO
- C805: footprint (none) -> P800_footprint_library:cap_electrolytic_UFG1H101MPM1TD
- C806: footprint (none) -> Capacitor_THT:C_Rect_L13.0mm_W5.0mm_P10.00mm_FKS3_FKP3_MKS4
- C807: footprint (none) -> P800_footprint_library:cap_ceramic_RCER71H473K0M1H03A
- C808: footprint (none) -> P800_footprint_library:cap_electrolytic_panasonic_5X11
- C809: footprint (none) -> P800_footprint_library:cap_electrolytic_UFG1C471MPM1TD
- F1: footprint (none) -> P800_footprint_library:fuse_holder_0PTF0078P
- H805: footprint (none) -> Package_TO_SOT_THT:TO-220-3_Vertical
- H806: footprint (none) -> Package_TO_SOT_THT:TO-92_Wide
- H807: footprint (none) -> Diode_THT:D_DO-41_SOD81_P10.16mm_Horizontal
- J2, J3, J4, J5: footprint P800_footprint_library:GRADCONN_RFPC-SMA27-F -> P800_footprint_library:sma_connector_RFPC-SMA27-F
- R801, R805: footprint (none) -> Resistor_SMD:R_2512_6332Metric_Pad1.40x3.35mm_HandSolder
- R803, R804, R806, R807: footprint (none) -> Resistor_SMD:R_1206_3216Metric_Pad1.30x1.75mm_HandSolder
- R808: footprint (none) -> P800_footprint_library:pot_3386F-1-502LF
Connections:
- net GND: now also HS1.1
Changed lines of the file:
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@@
 			)
 		)
-		(property "Footprint" "P800_footprint_library:GRADCONN_RFPC-SMA27-F"
+		(property "Footprint" "P800_footprint_library:sma_connector_RFPC-SMA27-F"
 			(at 215.9 83.82 0)
 			(effects
@@
 			)
 		)
-		(property "Footprint" ""
+		(property "Footprint" "Package_TO_SOT_THT:TO-92_Wide"
 			(at 165.1 100.33 0)
 			(effects
@@
 			)
 		)
-		(property "Footprint" ""
+		(property "Footprint" "P800_footprint_library:cap_electrolytic_UFG1H101MPM1TD"
 			(at 130.81 114.3 0)
 			(effects
@@
 			)
 		)
-		(property "Footprint" ""
+		(property "Footprint" "P800_footprint_library:cap_electrolytic_UKW1J471MHD1TO"
 			(at 121.92 114.3 0)
 			(effects
@@
 				(path "/0d9326c1-41e9-4c7f-81ed-9b5d802cb1b5"
 					(reference "C804")
+					(unit 1)
+				)
+			)
+		)
+	)
+	(symbol
+		(lib_id "Mechanical:Heatsink_Pad")
+		(at 39.37 97.79 0)
+		(unit 1)
+		(exclude_from_sim yes)
+		(in_bom yes)
+		(on_board yes)
+		(dnp no)
+		(property "Reference" "HS1"
+			(at 38.1 93.98 0)
+			(effects
+				(font
+					(size 1.27 1.27)
+				)
+				(justify left)
+			)
+		)
+		(property "Value" "Heatsink_Pad"
+			(at 43.18 98.4249 0)
+			(effects
+				(font
+					(size 1.27 1.27)
+				)
+				(justify left)
+				(hide yes)
+			)
+		)
+		(property "Footprint" "P800_footprint_library:heatsink_577202B04000G"
+			(at 39.6748 99.06 0)
+			(effects
+				(font
+					(size 1.27 1.27)
+				)
+				(hide yes)
+			)
+		)
+		(property "Datasheet" "~"
+			(at 39.6748 99.06 0)
+			(effects
+				(font
+					(size 1.27 1.27)
+				)
+				(hide yes)
+			)
+		)
+		(property "Description" "Heatsink with electrical connection, 1 pin"
+			(at 39.37 97.79 0)
+			(effects
+				(font
+					(size 1.27 1.27)
+				)
+				(hide yes)
+			)
+		)
+		(pin "1"
+		)
+		(instances
+			(project ""
+				(path "/0d9326c1-41e9-4c7f-81ed-9b5d802cb1b5"
+					(reference "HS1")
 					(unit 1)
 				)
@@
 			)
 		)
-		(property "Footprint" ""
+		(property "Footprint" "Resistor_SMD:R_1206_3216Metric_Pad1.30x1.75mm_HandSolder"
 			(at 193.294 89.916 90)
 			(effects
@@
 			)
 		)
-		(property "Footprint" ""
+		(property "Footprint" "P800_footprint_library:fuse_holder_0PTF0078P"
 			(at 60.96 76.708 90)
 			(effects
@@
 			)
 		)
-		(property "Footprint" ""
+		(property "Footprint" "P800_footprint_library:cap_electrolytic_panasonic_5X11"
 			(at 179.07 90.17 0)
 			(effects
@@
 			)
 		)
-		(property "Footprint" ""
+		(property "Footprint" "P800_footprint_library:cap_electrolytic_A50"
 			(at 181.61 72.39 0)
 			(effects
@@
 			)
 		)
-		(property "Footprint" ""
+		(property "Footprint" "P800_footprint_library:cap_electrolytic_UFG1C471MPM1TD"
 			(at 180.34 118.11 0)
 			(effects
@@
 			)
 		)
-		(property "Footprint" ""
+		(property "Footprint" "Package_TO_SOT_THT:TO-220-3_Vertical"
 			(at 140.97 81.28 0)
 			(effects
@@
 			)
 		)
-		(property "Footprint" "P800_footprint_library:GRADCONN_RFPC-SMA27-F"
+		(property "Footprint" "P800_footprint_library:sma_connector_RFPC-SMA27-F"
 			(at 215.9 110.49 0)
 			(effects
@@
 			)
 		)
-		(property "Footprint" ""
+		(property "Footprint" "Diode_THT:D_DO-41_SOD81_P10.16mm_Horizontal"
 			(at 167.64 118.11 0)
 			(effects
@@
 			)
 		)
-		(property "Footprint" "P800_footprint_library:GRADCONN_RFPC-SMA27-F"
+		(property "Footprint" "P800_footprint_library:sma_connector_RFPC-SMA27-F"
 			(at 215.9 53.34 0)
 			(effects
@@
 			)
 		)
-		(property "Footprint" ""
+		(property "Footprint" "Capacitor_THT:C_Rect_L13.0mm_W5.0mm_P10.00mm_FKS3_FKP3_MKS4"
 			(at 144.4752 118.11 0)
 			(effects
@@
 			)
 		)
-		(property "Footprint" ""
+		(property "Footprint" "P800_footprint_library:cap_electrolytic_UKW1J471MHD1TO"
 			(at 113.03 114.3 0)
 			(effects
@@
 			)
 		)
-		(property "Footprint" ""
+		(property "Footprint" "P800_footprint_library:pot_3386F-1-502LF"
 			(at 194.31 102.87 0)
 			(effects
@@
 			)
 		)
-		(property "Footprint" ""
+		(property "Footprint" "P800_footprint_library:cap_ceramic_RCER71H473K0M1H03A"
 			(at 155.9052 119.38 0)
 			(effects
@@
 			)
 		)
-		(property "Footprint" "P800_footprint_library:GRADCONN_RFPC-SMA27-F"
+		(property "Footprint" "P800_footprint_library:sma_connector_RFPC-SMA27-F"
 			(at 215.9 68.58 0)
 			(effects
@@
 			)
 		)
-		(property "Footprint" ""
+		(property "Footprint" "P800_footprint_library:cap_electrolytic_A50"
 			(at 181.61 57.15 0)
 			(effects
@@
 			)
 		)
-		(property "Footprint" ""
+		(property "Footprint" "P800_footprint_library:cap_ceramic_RDER72H103K1M1H03A"
 			(at 70.8152 87.63 0)
 			(effects
@@
 			)
 		)
-		(property "Footprint" ""
+		(property "Footprint" "Resistor_SMD:R_1206_3216Metric_Pad1.30x1.75mm_HandSolder"
 			(at 136.906 97.536 90)
 			(effects
@@
 			)
 		)
-		(property "Footprint" ""
+		(property "Footprint" "Resistor_SMD:R_2512_6332Metric_Pad1.40x3.35mm_HandSolder"
 			(at 153.924 89.916 90)
 			(effects
@@
 			)
 		)
-		(property "Footprint" ""
+		(property "Footprint" "Resistor_SMD:R_2512_6332Metric_Pad1.40x3.35mm_HandSolder"
 			(at 117.094 82.804 90)
 			(effects
@@
 			)
 		)
-		(property "Footprint" ""
+		(property "Footprint" "Resistor_SMD:R_1206_3216Metric_Pad1.30x1.75mm_HandSolder"
 			(at 193.294 116.586 90)
 			(effects
@@
 	)
 	(symbol
+		(lib_id "power:GND")
+		(at 39.37 100.33 0)
+		(unit 1)
+		(exclude_from_sim no)
+		(in_bom yes)
+		(on_board yes)
+		(dnp no)
+		(fields_autoplaced yes)
+		(property "Reference" "#PWR07"
+			(at 39.37 106.68 0)
+			(effects
+				(font
+					(size 1.27 1.27)
+				)
+				(hide yes)
+			)
+		)
+		(property "Value" "GND"
+			(at 39.37 105.41 0)
+			(effects
+				(font
+					(size 1.27 1.27)
+				)
+				(hide yes)
+			)
+		)
+		(property "Footprint" ""
+			(at 39.37 100.33 0)
+			(effects
+				(font
+					(size 1.27 1.27)
+				)
+				(hide yes)
+			)
+		)
+		(property "Datasheet" ""
+			(at 39.37 100.33 0)
+			(effects
+				(font
+					(size 1.27 1.27)
+				)
+				(hide yes)
+			)
+		)
+		(property "Description" "Power symbol creates a global label with name \"GND\" , ground"
+			(at 39.37 100.33 0)
+			(effects
+				(font
+					(size 1.27 1.27)
+				)
+				(hide yes)
+			)
+		)
+		(pin "1"
+		)
+		(instances
+			(project ""
+				(path "/0d9326c1-41e9-4c7f-81ed-9b5d802cb1b5"
+					(reference "#PWR07")
+					(unit 1)
+				)
+			)
+		)
+	)
+	(symbol
 		(lib_id "Device:R_US")
 		(at 130.81 90.17 180)
@@
 			)
 		)
-		(property "Footprint" ""
+		(property "Footprint" "Resistor_SMD:R_1206_3216Metric_Pad1.30x1.75mm_HandSolder"
 			(at 129.794 89.916 90)
 			(effects
